File: kicad_sc11bbm/sc11bbm.kicad_sch (KiCad schematic)
At the start: 8 parts

Commit message: Update sc11bbm.kicad_sch
Parts:
- removed U?: BME280, symbol BME280:BME280
- added D?: LED, symbol Device:LED
- added R?: R, symbol Device:R
Connections:
- net GND: now also U?.2 (GND), U?.7 (GND), U?.8 (GND)
- net +5V: now reaches U?.1 (5V)
- net at U?.3 (RXD): now also D?.2 (A)
- net GPS4_1: now reaches U?.4 (TXD)
- net GPS4_1: now also A?.1 (D1/TX)
- net at A?.17 (3V3), U?.1 (+V), U?.1 (VCC): now also U?.8 (VDD), R?.1
- net at A?.16 (D13), U?.2 (SCL): now also U?.4 (SCK)
- net at A?.14 (D11), U?.3 (SDA): now also U?.3 (SDI)
- net at A?.15 (D12), U?.4 (SA0): now also U?.5 (SDO)
- net BME2_13: now reaches A?.13 (D10), U?.5 (CS)
- net BME2_13: now also U?.2 (CSB)
- net at A?.2 (D0/RX): now also D?.1 (K), R?.2
- no-connect marks 1 -> 6

Commit message: Update sc11bbm.kicad_sch
Parts:
- added U?: AE-MICRO-SD-DIP, symbol AE-MICRO-SD-DIP:AE-MICRO-SD-DIP
Connections:
- net BME2_13: now also U?.2 (DAT3)
- net at A?.16 (D13), U?.2 (SCL), U?.4 (SCK): now also U?.5 (CLK)
- net at A?.14 (D11), U?.3 (SDA), U?.3 (SDI): now also U?.3 (CMD)
- net at A?.15 (D12), U?.4 (SA0), U?.5 (SDO): now also U?.7 (DAT0)
- no-connect marks 6 -> 12
Other:
- moved on the sheet: U?
Changed lines of the file:
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@@
   (junction (at 132.08 64.77) (diameter 0) (color 0 0 0 0)
   )
+  (junction (at 114.3 105.41) (diameter 0) (color 0 0 0 0)
+  )
+  (junction (at 106.68 110.49) (diameter 0) (color 0 0 0 0)
+  )
   (junction (at 46.99 96.52) (diameter 0) (color 0 0 0 0)
   )
@@
   (junction (at 149.86 69.85) (diameter 0) (color 0 0 0 0)
   )
+  (junction (at 111.76 107.95) (diameter 0) (color 0 0 0 0)
+  )
+  (junction (at 109.22 113.03) (diameter 0) (color 0 0 0 0)
+  )
   (no_connect (at 201.93 74.93))
+  (no_connect (at 204.47 91.44))
+  (no_connect (at 204.47 83.82))
   (no_connect (at 64.77 82.55))
   (no_connect (at 64.77 80.01))
@@
   (no_connect (at 66.04 114.3))
   (no_connect (at 60.96 160.02))
-  (wire (pts (xy 104.14 113.03) (xy 116.84 113.03))
-    (stroke (width 0) (type default) (color 0 0 0 0))
-  )
+  (no_connect (at 204.47 106.68))
+  (no_connect (at 204.47 96.52))
+  (no_connect (at 204.47 101.6))
+  (no_connect (at 204.47 104.14))
   (wire (pts (xy 44.45 118.11) (xy 44.45 100.33))
     (stroke (width 0) (type default) (color 0 0 0 0))
@@
     (stroke (width 0) (type default) (color 0 0 0 0))
   )
+  (wire (pts (xy 106.68 110.49) (xy 106.68 134.62))
+    (stroke (width 0) (type default) (color 0 0 0 0))
+  )
   (wire (pts (xy 134.62 46.99) (xy 134.62 69.85))
     (stroke (width 0) (type default) (color 0 0 0 0))
@@
     (stroke (width 0) (type default) (color 0 0 0 0))
   )
+  (wire (pts (xy 109.22 113.03) (xy 116.84 113.03))
+    (stroke (width 0) (type default) (color 0 0 0 0))
+  )
   (wire (pts (xy 49.53 64.77) (xy 93.98 64.77))
     (stroke (width 0) (type default) (color 0 0 0 0))
@@
     (stroke (width 0) (type default) (color 0 0 0 0))
   )
-  (wire (pts (xy 110.49 107.95) (xy 116.84 107.95))
+  (wire (pts (xy 162.56 86.36) (xy 162.56 121.92))
     (stroke (width 0) (type default) (color 0 0 0 0))
   )
@@
     (stroke (width 0) (type default) (color 0 0 0 0))
   )
+  (wire (pts (xy 109.22 130.81) (xy 168.91 130.81))
+    (stroke (width 0) (type default) (color 0 0 0 0))
+  )
   (wire (pts (xy 101.6 106.68) (xy 101.6 64.77))
     (stroke (width 0) (type default) (color 0 0 0 0))
@@
     (stroke (width 0) (type default) (color 0 0 0 0))
   )
+  (wire (pts (xy 111.76 107.95) (xy 111.76 127))
+    (stroke (width 0) (type default) (color 0 0 0 0))
+  )
   (wire (pts (xy 99.06 91.44) (xy 106.68 91.44))
     (stroke (width 0) (type default) (color 0 0 0 0))
@@
     (stroke (width 0) (type default) (color 0 0 0 0))
   )
-  (wire (pts (xy 113.03 105.41) (xy 116.84 105.41))
-    (stroke (width 0) (type default) (color 0 0 0 0))
-  )
   (wire (pts (xy 101.6 64.77) (xy 132.08 64.77))
     (stroke (width 0) (type default) (color 0 0 0 0))
@@
     (stroke (width 0) (type default) (color 0 0 0 0))
   )
+  (wire (pts (xy 111.76 107.95) (xy 116.84 107.95))
+    (stroke (width 0) (type default) (color 0 0 0 0))
+  )
   (wire (pts (xy 48.26 118.11) (xy 44.45 118.11))
     (stroke (width 0) (type default) (color 0 0 0 0))
@@
     (stroke (width 0) (type default) (color 0 0 0 0))
   )
+  (wire (pts (xy 111.76 127) (xy 165.1 127))
+    (stroke (width 0) (type default) (color 0 0 0 0))
+  )
+  (wire (pts (xy 165.1 88.9) (xy 204.47 88.9))
+    (stroke (width 0) (type default) (color 0 0 0 0))
+  )
   (wire (pts (xy 66.04 118.11) (xy 99.06 118.11))
     (stroke (width 0) (type default) (color 0 0 0 0))
@@
     (stroke (width 0) (type default) (color 0 0 0 0))
   )
+  (wire (pts (xy 106.68 134.62) (xy 172.72 134.62))
+    (stroke (width 0) (type default) (color 0 0 0 0))
+  )
   (wire (pts (xy 66.04 54.61) (xy 149.86 54.61))
     (stroke (width 0) (type default) (color 0 0 0 0))
   )
+  (wire (pts (xy 168.91 130.81) (xy 168.91 93.98))
+    (stroke (width 0) (type default) (color 0 0 0 0))
+  )
   (wire (pts (xy 93.98 80.01) (xy 93.98 143.51))
     (stroke (width 0) (type default) (color 0 0 0 0))
@@
     (stroke (width 0) (type default) (color 0 0 0 0))
   )
+  (wire (pts (xy 110.49 107.95) (xy 111.76 107.95))
+    (stroke (width 0) (type default) (color 0 0 0 0))
+  )
   (wire (pts (xy 149.86 69.85) (xy 201.93 69.85))
     (stroke (width 0) (type default) (color 0 0 0 0))
@@
     (stroke (width 0) (type default) (color 0 0 0 0))
   )
+  (wire (pts (xy 114.3 105.41) (xy 114.3 121.92))
+    (stroke (width 0) (type default) (color 0 0 0 0))
+  )
+  (wire (pts (xy 109.22 113.03) (xy 109.22 130.81))
+    (stroke (width 0) (type default) (color 0 0 0 0))
+  )
+  (wire (pts (xy 114.3 105.41) (xy 116.84 105.41))
+    (stroke (width 0) (type default) (color 0 0 0 0))
+  )
   (wire (pts (xy 158.75 113.03) (xy 142.24 113.03))
     (stroke (width 0) (type default) (color 0 0 0 0))
@@
     (stroke (width 0) (type default) (color 0 0 0 0))
   )
+  (wire (pts (xy 165.1 127) (xy 165.1 88.9))
+    (stroke (width 0) (type default) (color 0 0 0 0))
+  )
   (wire (pts (xy 48.26 114.3) (xy 46.99 114.3))
     (stroke (width 0) (type default) (color 0 0 0 0))
@@
     (stroke (width 0) (type default) (color 0 0 0 0))
   )
+  (wire (pts (xy 172.72 134.62) (xy 172.72 99.06))
+    (stroke (width 0) (type default) (color 0 0 0 0))
+  )
+  (wire (pts (xy 162.56 86.36) (xy 204.47 86.36))
+    (stroke (width 0) (type default) (color 0 0 0 0))
+  )
   (wire (pts (xy 93.98 64.77) (xy 101.6 64.77))
     (stroke (width 0) (type default) (color 0 0 0 0))
@@
     (stroke (width 0) (type default) (color 0 0 0 0))
   )
+  (wire (pts (xy 104.14 113.03) (xy 109.22 113.03))
+    (stroke (width 0) (type default) (color 0 0 0 0))
+  )
   (wire (pts (xy 66.04 46.99) (xy 134.62 46.99))
     (stroke (width 0) (type default) (color 0 0 0 0))
@@
     (stroke (width 0) (type default) (color 0 0 0 0))
   )
+  (wire (pts (xy 168.91 93.98) (xy 204.47 93.98))
+    (stroke (width 0) (type default) (color 0 0 0 0))
+  )
   (wire (pts (xy 93.98 76.2) (xy 93.98 80.01))
     (stroke (width 0) (type default) (color 0 0 0 0))
@@
   )
   (wire (pts (xy 66.04 49.53) (xy 158.75 49.53))
+    (stroke (width 0) (type default) (color 0 0 0 0))
+  )
+  (wire (pts (xy 172.72 99.06) (xy 204.47 99.06))
+    (stroke (width 0) (type default) (color 0 0 0 0))
+  )
+  (wire (pts (xy 113.03 105.41) (xy 114.3 105.41))
+    (stroke (width 0) (type default) (color 0 0 0 0))
+  )
+  (wire (pts (xy 114.3 121.92) (xy 162.56 121.92))
     (stroke (width 0) (type default) (color 0 0 0 0))
   )
@@
     (pin "1")
   )
+  (symbol (lib_id "AE-MICRO-SD-DIP:AE-MICRO-SD-DIP") (at 217.17 77.47 0) (unit 1)
+    (in_bom yes) (on_board yes) (fields_autoplaced)
+    (property "Reference" "U?" (id 0) (at 222.25 93.9799 0)
+      (effects (font (size 1.27 1.27)) (justify left))
+    )
+    (property "Value" "AE-MICRO-SD-DIP" (id 1) (at 222.25 96.5199 0)
+      (effects (font (size 1.27 1.27)) (justify left))
+    )
+    (property "Footprint" "" (id 2) (at 217.17 77.47 0)
+      (effects (font (size 1.27 1.27)) hide)
+    )
+    (property "Datasheet" "" (id 3) (at 217.17 77.47 0)
+      (effects (font (size 1.27 1.27)) hide)
+    )
+    (pin "1")
+    (pin "10")
+    (pin "2")
+    (pin "3")
+    (pin "4")
+    (pin "5")
+    (pin "6")
+    (pin "7")
+    (pin "8")
+    (pin "9")
+  )
   (symbol (lib_id "QMC5883L:QMC5883L") (at 210.82 59.69 0) (unit 1)
     (in_bom yes) (on_board yes) (fields_autoplaced)
@@
     (pin "1")
   )
-  (symbol (lib_id "Twe-Lite Red:Twe-Lite_Red") (at 223.52 105.41 0) (unit 1)
-    (in_bom yes) (on_board yes) (fields_autoplaced)
-    (property "Reference" "U?" (id 0) (at 254 108.9912 0))
-    (property "Value" "Twe-Lite_Red" (id 1) (at 254 111.5312 0))
-    (property "Footprint" "" (id 2) (at 223.52 105.41 0)
-      (effects (font (size 1.27 1.27)) hide)
-    )
-    (property "Datasheet" "" (id 3) (at 223.52 105.41 0)
+  (symbol (lib_id "Twe-Lite Red:Twe-Lite_Red") (at 227.33 109.22 0) (unit 1)
+    (in_bom yes) (on_board yes) (fields_autoplaced)
+    (property "Reference" "U?" (id 0) (at 257.81 112.8012 0))
+    (property "Value" "Twe-Lite_Red" (id 1) (at 257.81 115.3412 0))
+    (property "Footprint" "" (id 2) (at 227.33 109.22 0)
+      (effects (font (size 1.27 1.27)) hide)
+    )
+    (property "Datasheet" "" (id 3) (at 227.33 109.22 0)
       (effects (font (size 1.27 1.27)) hide)
     )
@@
       (reference "U?") (unit 1) (value "AE-GYSFDMAXB") (footprint "")
     )
+    (path "/5a84ce7b-5167-4eb2-aa6a-4df94f58a417"
+      (reference "U?") (unit 1) (value "AE-MICRO-SD-DIP") (footprint "")
+    )
     (path "/5faa8526-6821-49cd-a56c-914820a243cf"
